Commit message: update

File: isaacLab/manipulation/assets/urdf/kinova_robotiq/urdf/kinova_robotiq.urdf (robot description, URDF)
Before this commit: robot kinova_robotiq, 25 links, 24 joints
Links:
- link arm_base_link: geometry collision mesh filename=package://kinova_robotiq/meshes/collision/base_link.STL; visual mesh filename=package://kinova_robotiq/meshes/visual/base_link.STL
- link bracelet_link: geometry collision mesh filename=package://kinova_robotiq/meshes/collision/bracelet_with_vis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; visual mesh filename=package://kinova_robotiq/meshes/visual/bracelet_with_vision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
- link forearm_link: geometry collision mesh filename=package://kinova_robotiq/meshes/collision/forearm_link.STL; visual mesh filename=package://kinova_robotiq/meshes/visual/forearm_link.STL
- link half_arm_1_link: geometry collision mesh filename=package://kinova_robotiq/meshes/collision/half_arm_1_link.S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; visual mesh filename=package://kinova_robotiq/meshes/visual/half_arm_1_link.STL
- link half_arm_2_link: geometry collision mesh filename=package://kinova_robotiq/meshes/collision/half_arm_2_link.S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; visual mesh filename=package://kinova_robotiq/meshes/visual/half_arm_2_link.STL
- link left_inner_finger: geometry collision mesh filename=package://kinova_robotiq/meshes/collision/robotiq_arg2f_85_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 scale=0.001 0.001 0.001; visual mesh filename=package://kinova_robotiq/meshes/visual/robotiq_arg2f_85_inn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 scale=0.001 0.001 0.001
- link left_inner_knuckle: geometry collision mesh filename=package://kinova_robotiq/meshes/collision/robotiq_arg2f_85_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 scale=0.001 0.001 0.001; visual mesh filename=package://kinova_robotiq/meshes/visual/robotiq_arg2f_85_inn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 scale=0.001 0.001 0.001
- link left_outer_finger: geometry collision mesh filename=package://kinova_robotiq/meshes/collision/robotiq_arg2f_85_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 scale=0.001 0.001 0.001; visual mesh filename=package://kinova_robotiq/meshes/visual/robotiq_arg2f_85_out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 scale=0.001 0.001 0.001
- link left_outer_knuckle: geometry collision mesh filename=package://kinova_robotiq/meshes/collision/robotiq_arg2f_85_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 scale=0.001 0.001 0.001; visual mesh filename=package://kinova_robotiq/meshes/visual/robotiq_arg2f_85_out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 scale=0.001 0.001 0.001
- link right_inner_finger: geometry collision mesh filename=package://kinova_robotiq/meshes/collision/robotiq_arg2f_85_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 scale=0.001 0.001 0.001; visual mesh filename=package://kinova_robotiq/meshes/visual/robotiq_arg2f_85_inn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 scale=0.001 0.001 0.001
- link right_inner_knuckle: geometry collision mesh filename=package://kinova_robotiq/meshes/collision/robotiq_arg2f_85_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 scale=0.001 0.001 0.001; visual mesh filename=package://kinova_robotiq/meshes/visual/robotiq_arg2f_85_inn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 scale=0.001 0.001 0.001
- link right_outer_finger: geometry collision mesh filename=package://kinova_robotiq/meshes/collision/robotiq_arg2f_85_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 scale=0.001 0.001 0.001; visual mesh filename=package://kinova_robotiq/meshes/visual/robotiq_arg2f_85_out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 scale=0.001 0.001 0.001
- link right_outer_knuckle: geometry collision mesh filename=package://kinova_robotiq/meshes/collision/robotiq_arg2f_85_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 scale=0.001 0.001 0.001; visual mesh filename=package://kinova_robotiq/meshes/visual/robotiq_arg2f_85_out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 scale=0.001 0.001 0.001
- link robotiq_arg2f_base_link: geometry collision mesh filename=package://kinova_robotiq/meshes/collision/robotiq_arg2f_bas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; visual mesh filename=package://kinova_robotiq/meshes/collision/robotiq_arg2f_bas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
- link shoulder_link: geometry collision mesh filename=package://kinova_robotiq/meshes/collision/shoulder_link.STL; visual mesh filename=package://kinova_robotiq/meshes/visual/shoulder_link.STL
- link spherical_wrist_1_link: geometry collision mesh filename=package://kinova_robotiq/meshes/collision/spherical_wrist_1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; visual mesh filename=package://kinova_robotiq/meshes/visual/spherical_wrist_1_li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
- link spherical_wrist_2_link: geometry collision mesh filename=package://kinova_robotiq/meshes/collision/spherical_wrist_2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; visual mesh filename=package://kinova_robotiq/meshes/visual/spherical_wrist_2_li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

Commit message: Update kinova_robotiq.urdf

File: isaacLab/manipulation/assets/urdf/kinova_robotiq/urdf/kinova_robotiq.urdf (robot description, URDF)
Before this commit: robot kinova_robotiq, 25 links, 24 joints
Joints:
- joint arm_wheel: origin xyz=0.0 0.0 0.0 rpy=-1.57 0.0 0.0 -> xyz=0.0 0.0 0.0 rpy=-1.57 0.0 3.14
